Commit message: ARTI-D1 new mesh: assets, slow-gait reference motions, cfg
Mesh redesign (motion_generator robots/arti_d1): ankle-to-sole +20 mm (trunk 0.226 -> 0.246 m above the
pelvis origin), foot 63 -> 160 g with a filleted sole (flat face +-40 x +-17 mm), arm joints -5 deg and
ankles -9 deg of travel per side (plate rest -18 -> -13 deg).

- URDF / USD / meshes copied from motion_generator.
- Reference: 1000 clips of the slow gait (2.4 s cycle, 0.8 s single support, walk_com_height 0.235 -> 0.255
  so the leg pose is unchanged) + standing clip 1000.json; gen_motions.py honours [min, max] bounds.
- Env cfg: default pose, action ranges, commands, gait clock, knee lift target, trunk / sole offsets,
  sole patch size, termination height 0.17, joint speed capped at the servo no-load speed.
- pt_to_onnx / analyze_robot_log / check_controller_obs: new default pose, limits and sole offsets.

The nominal gait table (ILC) for the new mesh follows in a separate commit.

Co-Authored-By: Claude Opus 5.5 <noreply@anthropic.com>

File: source/arti_d1/arti_d1/assets/models/arti_d1/arti_d1.urdf (robot description, URDF)
Before this commit: robot pocketbot_final_v4, 18 links, 17 joints
Links:
- link left_arm_plate: mass 0.0613667 -> 0.0606196
- link left_foot_link: mass 0.0627159 -> 0.15981
- link right_arm_plate: mass 0.0613667 -> 0.0606195
- link right_foot_link: mass 0.0627159 -> 0.15981
Joints:
- joint left_ankle: limit lower=-1.96273 upper=0.72508 effort=10.6 velocity=3.14 -> lower=-1.80565 upper=0.568 effort=10.6 velocity=3.14
- joint left_arm_m8: limit lower=-1.13446 upper=0.436332 effort=4.1 velocity=4.82 -> lower=-1.0472 upper=0.349066 effort=4.1 velocity=4.82; origin xyz=0.0248485 0.12358 0.252732 rpy=0 0 0 -> xyz=0.0248443 0.12358 0.272732 rpy=0 0 0
- joint left_arm_m8crank_plate: limit lower=-0.314159 upper=1.25664 effort=4.1 velocity=4.82 -> lower=-0.226893 upper=1.16937 effort=4.1 velocity=4.82
- joint left_foot_frame: origin xyz=0.0135624237 -0.024 -0.0393326454 rpy=0 0 0 -> xyz=0.0135599213 -0.024 -0.0593316689 rpy=0 0 0
- joint left_hip_yaw: origin xyz=0.00965371 0.035 0.261048 rpy=0 0 0 -> xyz=0.00964957 0.035 0.281048 rpy=0 0 0
- joint right_ankle: limit lower=-1.96273 upper=0.72508 effort=10.6 velocity=3.14 -> lower=-1.80565 upper=0.568 effort=10.6 velocity=3.14
- joint right_arm_m8: limit lower=-1.13446 upper=0.436332 effort=4.1 velocity=4.82 -> lower=-1.0472 upper=0.349066 effort=4.1 velocity=4.82; origin xyz=0.0248485 -0.12358 0.252732 rpy=0 0 0 -> xyz=0.0248443 -0.12358 0.272732 rpy=0 0 0
- joint right_arm_m8crank_plate: limit lower=-0.314159 upper=1.25664 effort=4.1 velocity=4.82 -> lower=-0.226893 upper=1.16937 effort=4.1 velocity=4.82
- joint right_foot_frame: origin xyz=0.0135624237 0.024 -0.039332653 rpy=0 0 0 -> xyz=0.0135599213 0.0240000019 -0.0593316765 rpy=0 0 0
- joint right_hip_yaw: origin xyz=0.00965371 -0.035 0.261048 rpy=0 0 0 -> xyz=0.00964957 -0.035 0.281048 rpy=0 0 0
- joint trunk_frame: origin xyz=0.00965371 0 0.226248 rpy=0 0 0 -> xyz=0.00964957 0 0.246248 rpy=0 0 0

Commit message: ARTI-D1: new URDF (hip_roll frame 0.15 rad inward), re-converted USD, regenerated reference; drop AWS automation
URDF (motion_generator e7c14e0): left/right hip_roll joint frame rpy -/+0.15 rad, pelvis +7.797 mm.

- USD: re-converted from that URDF with Isaac Lab scripts/tools/convert_urdf.py (URDF importer 3.0,
  --joint_stiffness 0 --joint_damping 0): arti_d1.usda + payloads/ replace arti_d1.usd + configuration/. Colliders
  are convex hulls on the mesh prims, so the in-memory 5.1-layout patches (dangling trunk visual, Newton mesh
  colliders) and spawn_arti_d1_usd are removed. Links are nested under Robot/Geometry: IMU prim path updated.
- Reference: 1000 clips + standing clip (phase 0.9588, weight 176), same gait.json and commands. Only the stance
  hip_roll changes (-/+0.17466 -> -/+0.02466) and the root z (0.01225 -> 0.00445); other joints, speeds, swing and
  action ranges are identical.
- cfg: default pose, init root z, trunk offset z 0.254045; pt_to_onnx fallback pose.
- ILC table (8 iters): joint err <= 0.4 deg, zero-action sole peak 19 / 18 mm.
- check_amp_consistency: exact on PhysX and Newton (toes 2.0e-4 / 2.5e-4 m).
- Removed docker/, .dockerignore, control/run.yaml, scripts/automation/ (training runs locally).

Co-Authored-By: Claude Opus 5.5 <noreply@anthropic.com>

File: source/arti_d1/arti_d1/assets/models/arti_d1/arti_d1.urdf (robot description, URDF)
Before this commit: robot arti_d1, 18 links, 17 joints
Joints:
- joint left_arm_m8: origin xyz=0.0248443 0.12358 0.272732 rpy=0 0 0 -> xyz=0.0248443 0.12358 0.280529 rpy=0 0 0
- joint left_hip_roll: origin xyz=-0.0295 0 -0.10025 rpy=0 0 0 -> xyz=-0.0295 0 -0.10025 rpy=-0.15 0 0
- joint left_hip_yaw: origin xyz=0.00964957 0.035 0.281048 rpy=0 0 0 -> xyz=0.00964957 0.035 0.288845 rpy=0 0 0
- joint right_arm_m8: origin xyz=0.0248443 -0.12358 0.272732 rpy=0 0 0 -> xyz=0.0248443 -0.12358 0.280529 rpy=0 0 0
- joint right_hip_roll: origin xyz=-0.0295 0 -0.10025 rpy=0 0 0 -> xyz=-0.0295 0 -0.10025 rpy=0.15 0 0
- joint right_hip_yaw: origin xyz=0.00964957 -0.035 0.281048 rpy=0 0 0 -> xyz=0.00964957 -0.035 0.288845 rpy=0 0 0
- joint trunk_frame: origin xyz=0.00964957 0 0.246248 rpy=0 0 0 -> xyz=0.00964957 0 0.254045 rpy=0 0 0
